File: PCB/calbi.sch (EAGLE design)
At the start: 0 parts

Commit message: Schematic for AD9835 finished
Parts:
- added C1: 10uF, SparkFun-Capacitors:CAP0603-CAP
- added C3, C5: 0.1uF, SparkFun-Capacitors:CAP0603-CAP
- added C4: 0.01uF, SparkFun-Capacitors:CAP0603-CAP
- added C6, C8: .1 uF, SparkFun-Capacitors:CAP0603-CAP
- added C7: .01 uF, SparkFun-Capacitors:CAP0603-CAP
- added FRAME1: FRAME-LEDGER, SparkFun-Aesthetics:FRAME-LEDGER
- added J$1: SMA_EDGE, SparkFun-Connectors:SMA_EDGE
- added R2: (no value), SparkFun-Passives:RESISTOR0603-RES
- added R4: 3.9 K, SparkFun-Passives:RESISTOR0603-RES
- added R6: 300, SparkFun-Passives:RESISTOR0603-RES
- added U$1: AD8400ARZ100-NDSOIC-8, calbi:AD8400ARZ100-NDSOIC-8
- added U$2: AD9835, calbi:AD9835
- added U1: LT3086MPT7, calbi:LT3086MPT7
Connections:
- new net 3.3V: C3.1, C4.2, C5.1, U$2.AVDD, U$2.DVDD
- new net GND: C3.2, C5.2, C6.1, C7.1, C8.2, J$1.GND@0, J$1.GND@1, J$1.GND@2, J$1.GND@3, R4.2, R6.1, U$2.AGND, U$2.DGND
- new net GND-ISO: C1.1, C1.2, R2.1, U1.!SHDN, U1.GND, U1.IN
- new net N$1: C7.2, U$2.REFOUT
- new net N$2: R2.2, U1.IMON/ILIM
- new net N$3: C8.1, J$1.SIGNAL, R6.2, U$2.IOUT
- new net N$4: C4.1, U$2.COMP
- new net N$7: C6.2, R4.1, U$2.FS_ADJ
