File: PCB/calbi.brd (EAGLE design)
At the start: 0 parts

Commit message: Fixed a couple of errors in the schematic. Layed out power. Going to meet on Wednesday at 3:30 to do the RF layout
Parts:
- added C1, C2: 10uF, SparkFun-Capacitors:0603-CAP
- added C10, C3, C5: 0.1uF, SparkFun-Capacitors:0603-CAP
- added C11, C6, C8, C9: .1 uF, SparkFun-Capacitors:0603-CAP
- added C12, C13: 1 uF, SparkFun-Capacitors:0603-CAP
- added C4: 0.01uF, SparkFun-Capacitors:0603-CAP
- added C7: .01 uF, SparkFun-Capacitors:0603-CAP
- added FRAME1: FRAME-LEDGER, SparkFun-Aesthetics:CREATIVE_COMMONS
- added J$1: SMA_EDGE, SparkFun-Connectors:SMA-EDGE
- added J1, J2: (no value), SparkFun-Connectors:SCREWTERMINAL-3.5MM-2
- added R1, R5, R8: 1k, SparkFun-Passives:0603-RES
- added R2: 0 ohm, SparkFun-Passives:0603-RES
- added R3, R7, R9: 2k, SparkFun-Passives:0603-RES
- added R4: 3.9 K, SparkFun-Passives:0603-RES
- added R6: 300, SparkFun-Passives:0603-RES
- added U$1: V_REG_LD1117VXX, SparkFun-PowerIC:78XXL
- added U$2: AD9835, calbi:TSSOP16
- added U$3: AD8400ARZ100-NDSOIC-8, calbi:SO08
- added U1: LT3086MPT7, calbi:TO220-7
- added U2: 33MHZ-OSCILLATOR, SparkFun-FreqCtrl:CRYSTAL-OSC-SMD-5X3.2
- added _1: TEENSY, calbi:TEENSY
Connections:
- new net +5V: C10.1, C12.1, C9.1, U$1.OUT, U$3.6, _1.+5V
- new net 3.3V: C13.1, C3.1, C4.2, C5.1, U$1.GND, U$2.15, U$2.4, U2.2, U2.4
- new net GND: C1.2, C10.2, C12.2, C13.2, C2.1, C3.2, C5.2, C6.1, C7.1, C8.2, C9.2, J$1.GND@0, J$1.GND@1, J$1.GND@2, J$1.GND@3, J1.1, J2.2, R2.1, R4.2, R6.1, U$1.IN, U$2.13, U$2.5, U$3.2, U1.4, _1.GND, _1.GRND1
- new net MOSI: R8.2, U$3.4, _1.B2
- new net MOSI3.3: R8.1, R9.2, U$2.8
- new net N$1: C7.2, U$2.3
- new net N$10: U$3.1, U1.2
- new net N$12: R7.1
- new net N$13: R9.1
- new net N$2: R2.2, U1.1
- new net N$3: C8.1, J$1.SIG, R6.2, U$2.14
- new net N$4: C4.1, U$2.16
- new net N$5: C2.2, J2.1, U$3.7, U1.3
- new net N$6: U$2.2, U2.3
- new net N$7: C6.2, R4.1, U$2.1
- new net N$8: C1.1, J1.2, U1.5
- new net N$9: R3.1
- new net SCLK: R5.2, U$3.5, _1.B1
- new net SCLK3.3: R5.1, R7.2, U$2.7
- new net \CS0: U$3.3, _1.B0
- new net \CS1: R1.2, _1.B7
- new net \CS13.3: R1.1, R3.2, U$2.9
- new net \SHDN: U1.6, _1.D0
Routing:
- net GND: track 0.00 -> 81.8 mm, vias 0 -> 1
- net +5V: track 0.00 -> 54.6 mm
- net N$5: track 0.00 -> 46.3 mm
- net N$8: track 0.00 -> 31.3 mm
- net N$10: track 0.00 -> 9.10 mm
- net 3.3V: track 0.00 -> 2.96 mm
- net N$11: track 0.00 -> 1.27 mm
Other:
- board outline added: 100 x 80 mm

Commit message: Commiting changes from Wednesday
Parts:
- C11: value .1 uF -> 0.1uF
- moved J$1 127.0 mm to (57.1, 15.6), turned to 90 degrees
- moved C3 126.1 mm to (46.4, 16.5), flipped to the bottom, turned to 270 degrees
- moved R4 116.7 mm to (42.2, 23.2), turned to 90 degrees
- moved C8 98.5 mm to (52.7, 17.1), turned to 270 degrees
- moved U2 98.1 mm to (37.1, 20.0), turned to 270 degrees
- moved C11 93.5 mm to (37.1, 20.0), flipped to the bottom, turned to 270 degrees
- moved R2 90.9 mm to (33.7, 73.0), flipped to the bottom, turned to 90 degrees
- moved R6 86.9 mm to (50.8, 17.1), turned to 90 degrees
- moved C7 86.0 mm to (40.0, 15.6), turned to 90 degrees
- moved C5 84.0 mm to (44.5, 14.9), flipped to the bottom, turned to 270 degrees
- moved C6 80.1 mm to (42.2, 23.2), flipped to the bottom, turned to 270 degrees
- moved C4 79.4 mm to (48.3, 22.2), turned to 90 degrees
- moved U$2 77.1 mm to (45.1, 17.1), turned to 270 degrees
- moved R3 60.8 mm to (71.8, 66.0)
- moved R9 60.8 mm to (81.9, 66.0)
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Connections:
- net 3.3V: now also C11.1; no longer U2.2
- net GND: now also C11.2, U2.2
Routing:
- net GND: track 81.8 -> 121.2 mm
- net N$3: track 0.00 -> 11.2 mm
- net 3.3V: track 2.96 -> 13.9 mm
- net N$7: track 0.00 -> 4.33 mm
- net N$6: track 0.00 -> 3.99 mm
- net N$2: track 0.00 -> 3.78 mm
- net N$1: track 0.00 -> 3.54 mm
- net +5V: track 54.6 -> 56.0 mm
- added copper zone on layer 16, net N$21

Commit message: FInished up a few things. Set up the cam.
Parts:
- moved R9 75.5 mm to (25.7, 15.6)
- moved R8 75.5 mm to (25.7, 19.4), turned to 90 degrees
- moved R3 70.1 mm to (23.2, 15.6)
- moved R1 70.1 mm to (23.2, 19.4)
- moved R7 70.1 mm to (28.3, 15.6)
- moved R5 70.1 mm to (28.3, 19.4)
- flipped C7 to the bottom
Connections:
- removed net N$12: R7.1
- removed net N$13: R9.1
- removed net N$9: R3.1
- net GND: now also R3.1, R7.1, R9.1
Routing:
- net GND: track 121.2 -> 347.7 mm, vias 1 -> 3
- net SCLK: track 0.00 -> 91.2 mm, vias 0 -> 2
- net MOSI: track 0.00 -> 90.7 mm, vias 0 -> 1
- net +5V: track 56.0 -> 139.5 mm, vias 0 -> 1
- net 3.3V: track 13.9 -> 68.1 mm, vias 0 -> 2
- net \CS1: track 0.00 -> 47.1 mm, vias 0 -> 1
- net \CS0: track 0.00 -> 43.1 mm
- net \CS13.3: track 0.00 -> 40.3 mm, vias 0 -> 2
- net \SHDN: track 0.00 -> 28.9 mm, vias 0 -> 1
- net MOSI3.3: track 0.00 -> 23.9 mm, vias 0 -> 3
- net SCLK3.3: track 0.00 -> 17.1 mm
- net N$1: track 3.54 -> 9.09 mm, vias 0 -> 1
- net N$7: track 4.33 -> 6.98 mm, vias 0 -> 1
- net N$4: track 0.00 -> 2.33 mm
- net N$3: track 11.2 -> 12.1 mm
- added copper zone on layer 16, net GND
- removed copper zone on layer 16, net N$21
Other:
- board size 100 x 80 mm -> 59 x 80 mm
